File: Electronics/Robot/Robot.brd (EAGLE design)
At the start: 160 x 100 mm, 0 parts

Commit message: Buzzer, Teensy 4.0 Robot
Parts:
- added C1: 100nF, rcl:C050-024X044
- added H1, H2, H3, H4: MOUNT-HOLE3.0, holes:3,0
- added JP1: B3B-PH-K-S, con-JST PH:B3B-PH-K-S
- added Q1, Q2: 2N7000, transistor-small-signal:SOT54E
- added R13, R14, R15, R16, R3: 10k, rcl:0207/10
- added R4: 2K2, rcl:0207/10
- added SG1: F/EE17P, buzzer:F/EE17P
- added T1: (no value), transistor:TO92-EBC
- added U$1: TEENSY_4.0, Teensy_3_and_LC_Series_Boards_v1.4:TEENSY_4.0
- added U$2, U$3: DYNAMIXEL_CONNECTOR_TTL, DYNAMIXEL_CONNECTOR_TTL:DYNAMIXEL_CONNECTOR_TTL
- added U$4: WIRELESS-BLUETOOTH-HC-05, TP4056:WIRELESS-BLUETOOTH-HC-05
- added U1: GY-521MPU6050, gy-521:GY-521
- added U2: SN74LS241N, SN74LS241N:DIP254P762X508-20
- added X1: (no value), con-wago-500:W237-102
Connections:
- new net +12V: U$2.VDD, U$3.VDD, X1.1
- new net +3V3: U$1.3V3, U$1.3V3_1, U1.VCC
- new net +5V: C1.1, R3.1, SG1.1, U$1.VIN, U$4.5, U2.20
- new net AGND: U$1.AGND
- new net BL_RX: Q1.S, R13.2, U$1.8
- new net BL_STATE: U$4.1
- new net BL_TX: Q2.S, R14.2, U$1.7
- new net BUZZER: R4.1, U$1.23
- new net DATA: R3.2, U$2.DATA, U$3.DATA, U2.2, U2.3
- new net ENABLE_AX12: U2.1, U2.19
- new net GND: C1.2, JP1.3, T1.E, U$1.GND, U$1.GND2, U$2.GND, U$3.GND, U$4.4, U1.GND, U2.10, X1.2
- new net GY_SCL: U$1.19, U1.SCL
- new net GY_SDA: U$1.18, U1.SDA
- new net N$1: Q1.G, Q2.G, R13.1, R14.1
- new net N$100: Q1.D, R15.2, U$4.2
- new net N$1001: Q2.D, R16.2, U$4.3
- new net N$3: R15.1, R16.1
- new net N$7: R4.2, T1.B
- new net N$8: SG1.2, T1.C
- new net RX_AX12: U2.18
- new net SSC-32-RX: JP1.2, U$1.14
- new net SSC-32-TX: JP1.1, U$1.15
- new net TX_AX12: U2.17
- new net VBAT: U$1.VBAT
Other:
- board size 160 x 100 mm -> 76.2 x 59.4 mm
