File: Electronics/Robot/Robot.sch (EAGLE design)
At the start: 0 parts

Commit message: Buzzer, Teensy 4.0 Robot
Parts:
- added C1: 100nF, rcl:C-EU050-024X044
- added H1, H2, H3, H4: MOUNT-HOLE3.0, holes:MOUNT-HOLE3.0
- added JP1: B3B-PH-K-S, con-JST PH:B3B-PH-K-S
- added Q1, Q2: 2N7000, transistor-small-signal:BS170
- added R13, R14, R15, R16, R3: 10k, rcl:R-EU_0207/10
- added R4: 2K2, rcl:R-EU_0207/10
- added SG1: F/EE17P, buzzer:F/EE17P
- added T1: (no value), transistor:-NPN-TO92-EBC
- added U$1: TEENSY_4.0, Teensy_3_and_LC_Series_Boards_v1.4:TEENSY_4.0
- added U$2, U$3: DYNAMIXEL_CONNECTOR_TTL, DYNAMIXEL_CONNECTOR_TTL:DYNAMIXEL_CONNECTOR_TTL
- added U$4: WIRELESS-BLUETOOTH-HC-05, TP4056:WIRELESS-BLUETOOTH-HC-05
- added U1: GY-521MPU6050, gy-521:GY-521MPU6050
- added U2: SN74LS241N, SN74LS241N:SN74LS241N
- added X1: (no value), con-wago-500:W237-102
Connections:
- new net +12V: U$2.VDD, U$3.VDD, X1-1.KL
- new net +3V3: U$1.3.3V, U1.VCC
- new net +5V: C1.1, R3.1, SG1.1, U$1.VIN, U$4.+5V, U2.VCC
- new net BL_RX: Q1.S, R13.2, U$1.8/TX2/PWM
- new net BL_STATE: U$4.STATE
- new net BL_TX: Q2.S, R14.2, U$1.7/RX2/PWM
- new net BUZZER: R4.1, U$1.23/A9/PWM
- new net DATA: R3.2, U$2.DATA, U$3.DATA, U2.1A1, U2.2Y4
- new net ENABLE_AX12: U2.1~G, U2.2G
- new net GND: C1.2, JP1.3, T1.E, U$1.GND, U$2.GND, U$3.GND, U$4.GND, U1.GND, U2.GND, X1-2.KL
- new net GY_SCL: U$1.19/A5/SCL0/PWM, U1.SCL
- new net GY_SDA: U$1.18/A4/SDA0/PWM, U1.SDA
- new net N$1: Q1.G, Q2.G, R13.1, R14.1
- new net N$100: Q1.D, R15.2, U$4.RX
- new net N$1001: Q2.D, R16.2, U$4.TX
- new net N$3: R15.1, R16.1
- new net N$7: R4.2, T1.B
- new net N$8: SG1.2, T1.C
- new net RX_AX12: U2.1Y1
- new net SSC-32-RX: JP1.2, U$1.14/A0/TX3/PWM
- new net SSC-32-TX: JP1.1, U$1.15/A1/RX3/PWM
- new net TX_AX12: U2.2A4
Other:
- note added: "Buzzer"
- note added: "Dynamixel Communication Circuit"
